Commit message: feat: publish Isaac ground-truth odometry to ROS 2

File: isaac_sim/assets/lekiwi_soarm/source_xacro/lekiwi_soarm.urdf.xacro (robot description, xacro)
@@ -36,5 +36,6 @@
     <parent link="base_footprint"/>
     <child link="base_link"/>
-    <origin xyz="0 0 0.055" rpy="0 0 0"/>
+    <!-- Put base_footprint on the nominal three-wheel ground-contact plane. -->
+    <origin xyz="0 0 0.075" rpy="0 0 0"/>
   </joint>
   <link name="base_link">
